Commit message: Actionlib_sample server and client fixed

File: bot/src/model/bot.xacro (robot description, xacro)
@@ -123,4 +123,30 @@
     <origin xyz="${bot_length/3} ${bot_width/2} ${-bot_height/2}" rpy="0 0 0"/>
   </xacro:wheel>
+  <!-- LIDAR -->
+  <joint name="lidar_joint" type="fixed">
+    <axis xyz="0 0 0" />
+    <origin xyz="${bot_length*6/7} 0 ${bot_height}" rpy="0 0 0"/>
+    <parent link="base_link"/>
+    <child link="lidar"/>
+  </joint>
+  <link name="lidar">
+    <collision>
+      <origin xyz="0 0 0" rpy="0 0 0"/>
+      <geometry>
+        <box size="0.03 0.03 0.03"/>
+      </geometry>
+    </collision>
+    <visual>
+      <origin xyz="0 0 0" rpy="0 0 0"/>
+      <geometry>
+        <box size="0.03 0.03 0.03"/>
+      </geometry>
+    </visual>
+    <inertial>
+      <mass value="1e-5" />
+      <origin xyz="0 0 0" rpy="0 0 0"/>
+      <inertia ixx="1e-6" ixy="0" ixz="0" iyy="1e-6" iyz="0" izz="1e-6" />
+    </inertial>
+  </link>
   <!-- GAZEBO PLUGINS -->
   <gazebo>
@@ -128,5 +154,5 @@
       <alwaysOn>true</alwaysOn>
       <publishTf>1</publishTf>
-      <updateRate>100</updateRate>
+      <updateRate>50</updateRate>
       <leftJoint>left_wheel_joint</leftJoint>
       <rightJoint>right_wheel_joint</rightJoint>
@@ -153,3 +179,39 @@
     <material>Gazebo/Red</material>
   </gazebo>
+  <gazebo reference="lidar">
+    <sensor type="ray" name="head_hokuyo_sensor_front">
+      <pose>0 0 0 0 0 0</pose>
+      <visualize>true</visualize>
+      <update_rate>40</update_rate>
+      <ray>
+        <scan>
+          <horizontal>
+            <samples>720</samples>
+            <resolution>1</resolution>
+            <min_angle>-1.3</min_angle>
+            <max_angle>1.3</max_angle>
+            <!-- 1.570796 -->
+          </horizontal>
+        </scan>
+        <range>
+          <min>0.1</min>
+          <max>30.0</max>
+          <resolution>0.01</resolution>
+        </range>
+        <noise>
+          <type>gaussian</type>
+          <!-- Noise parameters based on published spec for Hokuyo laser
+               achieving "+-30mm" accuracy at range < 10m.  A mean of 0.0m and
+               stddev of 0.01m will put 99.7% of samples within 0.03m of the true
+               reading. -->
+          <mean>0.0</mean>
+          <stddev>0.01</stddev>
+        </noise>
+      </ray>
+      <plugin name="gazebo_ros_head_hokuyo_controller" filename="libgazebo_ros_laser.so">
+        <topicName>scan</topicName>
+        <frameName>lidar</frameName>
+      </plugin>
+    </sensor>
+  </gazebo>
 </robot>

Commit message: Robot spinning upon reaching goal fixed

File: bot/src/model/bot.xacro (robot description, xacro)
@@ -20,4 +20,6 @@
     <inertia ixx="0.6" ixy="0" ixz="0" iyy="0.65" iyz="0" izz="0.21"/>
   </xacro:macro>
+<!-- BASE_FOOTPRINT PARAMETERS -->
+  <xacro:property name ="base_footprint_size" value="0.01"/>
 <!-- BALL PARAMETERS -->
   <xacro:property name="ball_radius" value="0.05"/>
@@ -30,4 +32,5 @@
   <xacro:property name="wheel_radius" value="${ball_radius}"/>
   <xacro:property name="wheel_thickness" value="0.02"/>
+  <xacro:property name="wheel_base_length_coefficient" value="${1/3}"/>
   <xacro:macro name="wheel_geometry">
     <geometry>
@@ -90,4 +93,30 @@
     </visual>
   </link>
+  <!-- BASE_FOOTPRINT -->
+  <link name='base_footprint'>
+    <collision name="base_footprint_collision">
+      <xacro:default_origin/>
+      <geometry>
+        <sphere radius="${base_footprint_size}"/>
+      </geometry>
+    </collision>
+    <visual name="ball_visual">
+      <xacro:default_origin/>
+      <geometry>
+        <sphere radius="${base_footprint_size}"/>
+      </geometry>
+    </visual>
+    <inertial>
+      <mass value="0.001"/>
+      <xacro:default_origin/>
+      <inertia ixx="0.0001" ixy="0" ixz="0" iyy="0.0001" iyz="0" izz="0.0001"/>
+    </inertial>
+  </link>
+  <joint type="fixed" name="base_ftprnt__base_link_joint">
+    <origin xyz="${bot_length*wheel_base_length_coefficient} 0 ${-bot_height/2}" rpy="0 0 0"/>
+    <child link="base_footprint"/>
+    <parent link="base_link"/>
+    <axis xyz="0 0 0" rpy="0 0 0"/>
+  </joint>
   <!-- CASTER BALL -->
   <link name="ball">
@@ -118,8 +147,8 @@
   <!-- WHEELS -->
   <xacro:wheel name="right">
-    <origin xyz="${bot_length/3} ${-bot_width/2} ${-bot_height/2}" rpy="0 0 0"/>
+    <origin xyz="${bot_length*wheel_base_length_coefficient} ${-bot_width/2} ${-bot_height/2}" rpy="0 0 0"/>
   </xacro:wheel>
   <xacro:wheel name="left">
-    <origin xyz="${bot_length/3} ${bot_width/2} ${-bot_height/2}" rpy="0 0 0"/>
+    <origin xyz="${bot_length*wheel_base_length_coefficient} ${bot_width/2} ${-bot_height/2}" rpy="0 0 0"/>
   </xacro:wheel>
   <!-- LIDAR -->
